File: CANRxPCB.kicad_sch (KiCad schematic)
At the start: 26 parts, among them CN1 8x2_FEM, CN2 10x2_FEM, CN3 15x2_FEM, CN4 17x2_FEM, J1 RLED_JST, J2 GLED_JST, J3 IO_CONN, J4 SW_CONN, J5 BTN_JST, SW1 2M1-SP1-T1-B1-M2QE, SW2 SW_Push, U1 12V_POK, U2 MICROSD_SDIO, U3 BxCAN, U4 RTCModule, U5 12Vto5V, U6 CAN_TRx

Commit message: Final PCB Version
Parts:
- removed R2, R3: R, Resistor_THT:R_Axial_DIN0207_L6.3mm_D2.5mm_P7.62mm_Horizontal, symbol Device:R
- added R1: R, Resistor_THT:R_Axial_DIN0207_L6.3mm_D2.5mm_P7.62mm_Horizontal, symbol Device:R
- U1: renamed from U5; value 12Vto5V -> 12Vto12V
- renumbered C4 to C1, C1 to C2, C2 to C3, C3 to C4, CN3 to CN2, CN2 to CN3, D2 to D1, D1 to D2, J3 to J1, J1 to J2, J2 to J3, J5 to J4, J4 to J5, R1 to R2, SW2 to SW1, SW1 to SW2, U6 to U2, U1 to U4, U2 to U5, U4 to U6
Connections:
- net +5V is gone; now on net +12V: C4.1, CN1.15, U1.1 (OUTPUT)
- net +12V: no longer C3.1, J1.1 (Pin_1), U1.3 (INPUT), U4.5 (VCC)
- net +3.3V: now also D1.2 (A), J2.1 (Pin_1)
- net GND: now also D2.1 (K), J3.2 (Pin_2)
- net PG0: now also R1.1; no longer D1.1 (K), D2.2 (A), J2.2 (Pin_2), J3.1 (Pin_1)
- new net: D1.1 (K), D2.2 (A), J2.2 (Pin_2), J3.1 (Pin_1), R1.2
- new net +12VA: C3.1, J1.1 (Pin_1), U1.3 (INPUT), U4.5 (VCC)
Other:
- moved on the sheet: D1, D2, J2, J3
